File: mosturePartBoard.kicad_sch (KiCad schematic)
At the start: 22 parts, among them J1 Conn_01x08_Pin, J2 Conn_01x08_Pin, J3 Conn_01x03_Pin, J4 Conn_01x02_Pin, P1 USB_C_Plug_USB2.0, U1 TP4056-42-ESOP8

Commit message: need to edit powerlines
Parts:
- removed P1: USB_C_Plug_USB2.0, Connector_USB:USB_C_Receptacle_GCT_USB4105-xx-A_16P_TopMnt_Horizontal, symbol Connector:USB_C_Plug_USB2.0
- J3: footprint Connector_PinHeader_2.54mm:PinHeader_1x03_P2.54mm_Vertical_SMD_Pin1Right -> Connector_PinHeader_2.54mm:PinHeader_1x03_P2.54mm_Vertical
- J4: footprint Connector_JST:JST_JWPF_B02B-JWPF-SK-R_1x02_P2.00mm_Vertical -> Connector_Molex:Molex_CLIK-Mate_502443-0270_1x02-1MP_P2.00mm_Vertical
Connections:
- net GND: now also J1.2 (Pin_2)
- net VVCC: now also J1.1 (Pin_1)
- no-connect marks 17 -> 11
Changed lines of the file:
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@@
 	(paper "A4")
 	(junction
-		(at 223.52 48.26)
-		(diameter 0)
-		(color 0 0 0 0)
-	)
-	(junction
 		(at 149.86 62.23)
 		(diameter 0)
@@
 	)
 	(no_connect
-		(at 254 71.12)
-	)
-	(no_connect
-		(at 243.84 71.12)
-	)
-	(no_connect
 		(at 189.23 78.74)
 	)
 	(no_connect
-		(at 248.92 71.12)
-	)
-	(no_connect
-		(at 60.96 67.31)
-	)
-	(no_connect
 		(at 189.23 71.12)
 	)
@@
 	)
 	(no_connect
-		(at 60.96 64.77)
-	)
-	(no_connect
 		(at 189.23 68.58)
 	)
@@
 	)
 	(no_connect
-		(at 256.54 71.12)
-	)
-	(no_connect
 		(at 60.96 74.93)
 	)
@@
 	(wire
 		(pts
-			(xy 213.36 48.26) (xy 223.52 48.26)
-		)
-		(stroke
-			(width 0)
-			(type default)
-		)
-	)
-	(wire
-		(pts
 			(xy 113.03 62.23) (xy 118.11 62.23)
 		)
@@
 	(wire
 		(pts
-			(xy 261.62 74.93) (xy 262.89 76.2)
-		)
-		(stroke
-			(width 0)
-			(type default)
-		)
-	)
-	(wire
-		(pts
 			(xy 189.23 111.76) (xy 199.39 111.76)
 		)
@@
 	(wire
 		(pts
-			(xy 180.34 116.84) (xy 181.61 116.84)
+			(xy 60.96 67.31) (xy 63.5 67.31)
 		)
 		(stroke
@@
 	(wire
 		(pts
-			(xy 173.99 111.76) (xy 181.61 111.76)
+			(xy 180.34 116.84) (xy 181.61 116.84)
 		)
 		(stroke
@@
 	(wire
 		(pts
-			(xy 180.34 116.84) (xy 180.34 121.92)
+			(xy 173.99 111.76) (xy 181.61 111.76)
 		)
 		(stroke
@@
 	(wire
 		(pts
-			(xy 223.52 48.26) (xy 223.52 55.88)
+			(xy 180.34 116.84) (xy 180.34 121.92)
 		)
 		(stroke
@@
 	(wire
 		(pts
-			(xy 261.62 71.12) (xy 261.62 74.93)
-		)
-		(stroke
-			(width 0)
-			(type default)
-		)
-	)
-	(wire
-		(pts
 			(xy 189.23 118.11) (xy 189.23 125.73)
 		)
@@
 		)
 	)
+	(wire
+		(pts
+			(xy 60.96 64.77) (xy 64.77 64.77)
+		)
+		(stroke
+			(width 0)
+			(type default)
+		)
+	)
 	(global_label "ADC"
 		(shape input)
@@
 	(global_label "VVCC"
 		(shape input)
-		(at 262.89 76.2 270)
+		(at 64.77 64.77 0)
 		(fields_autoplaced yes)
 		(effects
@@
 				(size 1.27 1.27)
 			)
-			(justify right)
+			(justify left)
 		)
 		(property "Intersheetrefs" "${INTERSHEET_REFS}"
-			(at 262.89 83.9024 90)
+			(at 72.4724 64.77 0)
 			(effects
 				(font
 					(size 1.27 1.27)
 				)
-				(justify right)
+				(justify left)
 				(hide yes)
 			)
@@
 			)
 		)
-		(property "Footprint" "Connector_PinHeader_2.54mm:PinHeader_1x03_P2.54mm_Vertical_SMD_Pin1Right"
+		(property "Footprint" "Connector_PinHeader_2.54mm:PinHeader_1x03_P2.54mm_Vertical"
 			(at 134.62 21.59 0)
 			(effects
@@
 	)
 	(symbol
+		(lib_id "power:GND")
+		(at 63.5 67.31 90)
+		(unit 1)
+		(exclude_from_sim no)
+		(in_bom yes)
+		(on_board yes)
+		(dnp no)
+		(fields_autoplaced yes)
+		(property "Reference" "#PWR06"
+			(at 69.85 67.31 0)
+			(effects
+				(font
+					(size 1.27 1.27)
+				)
+				(hide yes)
+			)
+		)
+		(property "Value" "GND"
+			(at 67.31 67.3099 90)
+			(effects
+				(font
+					(size 1.27 1.27)
+				)
+				(justify right)
+			)
+		)
+		(property "Footprint" ""
+			(at 63.5 67.31 0)
+			(effects
+				(font
+					(size 1.27 1.27)
+				)
+				(hide yes)
+			)
+		)
+		(property "Datasheet" ""
+			(at 63.5 67.31 0)
+			(effects
+				(font
+					(size 1.27 1.27)
+				)
+				(hide yes)
+			)
+		)
+		(property "Description" "Power symbol creates a global label with name \"GND\" , ground"
+			(at 63.5 67.31 0)
+			(effects
+				(font
+					(size 1.27 1.27)
+				)
+				(hide yes)
+			)
+		)
+		(pin "1"
+		)
+		(instances
+			(project "mosturePartBoard"
+				(path "/556a9975-40a0-40b5-ab85-081bc891b66b"
+					(reference "#PWR06")
+					(unit 1)
+				)
+			)
+		)
+	)
+	(symbol
 		(lib_id "Device:R")
 		(at 213.36 139.7 0)
@@
 	)
 	(symbol
-		(lib_id "power:GND")
-		(at 213.36 48.26 270)
-		(unit 1)
-		(exclude_from_sim no)
-		(in_bom yes)
-		(on_board yes)
-		(dnp no)
-		(fields_autoplaced yes)
-		(property "Reference" "#PWR011"
-			(at 207.01 48.26 0)
-			(effects
-				(font
-					(size 1.27 1.27)
-				)
-				(hide yes)
-			)
-		)
-		(property "Value" "GND"
-			(at 209.55 48.2599 90)
-			(effects
-				(font
-					(size 1.27 1.27)
-				)
-				(justify right)
-			)
-		)
-		(property "Footprint" ""
-			(at 213.36 48.26 0)
-			(effects
-				(font
-					(size 1.27 1.27)
-				)
-				(hide yes)
-			)
-		)
-		(property "Datasheet" ""
-			(at 213.36 48.26 0)
-			(effects
-				(font
-					(size 1.27 1.27)
-				)
-				(hide yes)
-			)
-		)
-		(property "Description" "Power symbol creates a global label with name \"GND\" , ground"
-			(at 213.36 48.26 0)
-			(effects
-				(font
-					(size 1.27 1.27)
-				)
-				(hide yes)
-			)
-		)
-		(pin "1"
-		)
-		(instances
-			(project "mosturePartBoard"
-				(path "/556a9975-40a0-40b5-ab85-081bc891b66b"
-					(reference "#PWR011")
-					(unit 1)
-				)
-			)
-		)
-	)
-	(symbol
 		(lib_id "Device:C")
 		(at 100.33 76.2 0)
@@
 			)
 		)
-		(property "Footprint" "Connector_JST:JST_JWPF_B02B-JWPF-SK-R_1x02_P2.00mm_Vertical"
+		(property "Footprint" "Connector_Molex:Molex_CLIK-Mate_502443-0270_1x02-1MP_P2.00mm_Vertical"
 			(at 242.57 128.27 0)
 			(effects
@@
 					(unit 1)
 				)
-			)
-		)
-	)
-	(symbol
-		(lib_id "Connector:USB_C_Plug_USB2.0")
-		(at 246.38 55.88 270)
-		(unit 1)
-		(exclude_from_sim no)
-		(in_bom yes)
-		(on_board yes)
-		(dnp no)
-		(fields_autoplaced yes)
-		(property "Reference" "P1"
-			(at 265.43 54.6099 90)
-			(effects
-				(font
-					(size 1.27 1.27)
-				)
-				(justify left)
-			)
-		)
-		(property "Value" "USB_C_Plug_USB2.0"
-			(at 265.43 57.1499 90)
-			(effects
-				(font
-					(size 1.27 1.27)
-				)
-				(justify left)
-			)
-		)
-		(property "Footprint" "Connector_USB:USB_C_Receptacle_GCT_USB4105-xx-A_16P_TopMnt_Horizontal"
-			(at 246.38 59.69 0)
-			(effects
-				(font
-					(size 1.27 1.27)
-				)
-				(hide yes)
-			)
-		)
-		(property "Datasheet" "https://www.usb.org/sites/default/files/documents/usb_type-c.zip"
-			(at 246.38 59.69 0)
-			(effects
-				(font
-					(size 1.27 1.27)
-				)
-				(hide yes)
-			)
-		)
-		(property "Description" "USB 2.0-only Type-C Plug connector"
-			(at 246.38 55.88 0)
-			(effects
-				(font
-					(size 1.27 1.27)
-				)
-				(hide yes)
-			)
-		)
-		(pin "B5"
-		)
-		(pin "B1"
-		)
-		(pin "B12"
-		)
-		(pin "A5"
-		)
-		(pin "A4"
-		)
-		(pin "A7"
-		)
-		(pin "A6"
-		)
-		(pin "A9"
-		)
-		(pin "B4"
-		)
-		(pin "A1"
-		)
-		(pin "B9"
-		)
-		(pin "S1"
-		)
-		(pin "A12"
-		)
-		(instances
-			(project ""
-				(path "/556a9975-40a0-40b5-ab85-081bc891b66b"
-					(reference "P1")
-					(unit 1)
-				)
