File: mosturePartBoard.kicad_pcb (KiCad board)
At the start: 2 copper layers, 18.1 x 24.9 mm, 22 parts, among them J1 Conn_01x08_Pin, J2 Conn_01x08_Pin, J3 Conn_01x03_Pin, J4 Conn_01x02_Pin, P1 USB_C_Plug_USB2.0, U1 TP4056-42-ESOP8

Commit message: need to edit powerlines
Parts:
- removed P1: USB_C_Plug_USB2.0, Connector_USB:USB_C_Receptacle_GCT_USB4105-xx-A_16P_TopMnt_Horizontal
- J3: footprint Connector_PinHeader_2.54mm:PinHeader_1x03_P2.54mm_Vertical_SMD_Pin1Right -> Connector_PinHeader_2.54mm:PinHeader_1x03_P2.54mm_Vertical
- J4: footprint Connector_JST:JST_JWPF_B02B-JWPF-SK-R_1x02_P2.00mm_Vertical -> Connector_Molex:Molex_CLIK-Mate_502443-0270_1x02-1MP_P2.00mm_Vertical
- moved J4 12.8 mm to (124.2, 45.5), turned to 0 degrees
- moved C4 8.43 mm to (122.2, 55.7), turned to 90 degrees
- moved R1 8.26 mm to (119.5, 62.4)
- moved C1 8.20 mm to (122.2, 57.6)
- moved C3 8.20 mm to (122.3, 62.2)
- moved L1 8.20 mm to (121.4, 57.6)
- moved PS1 8.20 mm to (120.7, 60.1)
- moved R2 8.20 mm to (129.0, 61.4)
- moved R5 8.20 mm to (129.0, 59.6)
- moved U1 8.20 mm to (125.8, 59.5)
- moved R3 8.20 mm to (129.0, 57.8)
- moved R4 8.20 mm to (125.5, 55.4)
- moved R6 8.20 mm to (127.3, 55.4)
- moved R7 8.20 mm to (129.0, 56.0)
- moved C2 8.14 mm to (119.5, 57.5)
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Connections:
- J1 pad 1: unconnected-(J1-Pin_1-Pad1) -> VVCC
- J1 pad 2: unconnected-(J1-Pin_2-Pad2) -> GND
Routing:
- net VBAT: track 13.0 -> 28.3 mm, vias 0 -> 2
- net Net-(D2-K): track 15.4 -> 23.7 mm, vias 2 -> 4
- net CTRL_SENS: track 14.8 -> 7.87 mm
- net LOAD: track 10.5 -> 15.7 mm
- net MAIN_PWR: track 23.5 -> 28.2 mm
- net VVCC: track 27.7 -> 23.1 mm, vias 3 -> 1
- net Net-(D1-K): track 13.6 -> 17.8 mm, vias 0 -> 2
- net ADC: track 13.9 -> 10.3 mm
- net Net-(U1-~{CHRG}): track 6.96 -> 8.65 mm, vias 0 -> 2
- net Net-(U1-CE): track 13.6 -> 13.0 mm
- net Net-(U1-~{STDBY}): track 7.22 -> 6.76 mm, vias 0 -> 2
- net GND: vias 4 -> 13
Other:
- board size 18.1 x 24.9 mm -> 18.1 x 23.5 mm

Commit message: restrusture
Parts:
- removed C3: 10u, Capacitor_SMD:C_0201_0603Metric_Pad0.64x0.40mm_HandSolder
- removed C4: 100n, Capacitor_SMD:C_0201_0603Metric_Pad0.64x0.40mm_HandSolder
- removed D2: LED, LED_SMD:LED_0201_0603Metric
- removed J4: Conn_01x02_Pin, Connector_Molex:Molex_CLIK-Mate_502443-0270_1x02-1MP_P2.00mm_Vertical
- removed R3: 10k, Resistor_SMD:R_0201_0603Metric_Pad0.64x0.40mm_HandSolder
- removed R4: 1k2, Resistor_SMD:R_0201_0603Metric_Pad0.64x0.40mm_HandSolder
- removed R5: 1k, Resistor_SMD:R_0201_0603Metric_Pad0.64x0.40mm_HandSolder
- removed R6: 4k7, Resistor_SMD:R_0201_0603Metric_Pad0.64x0.40mm_HandSolder
- removed R7: 47k, Resistor_SMD:R_0201_0603Metric_Pad0.64x0.40mm_HandSolder
- removed R8: R, Resistor_SMD:R_0201_0603Metric_Pad0.64x0.40mm_HandSolder
- removed U1: TP4056-42-ESOP8, Package_SO:SOIC-8-1EP_3.9x4.9mm_P1.27mm_EP2.41x3.3mm_ThermalVias
- added C5: 4u7, Capacitor_SMD:C_0201_0603Metric_Pad0.64x0.40mm_HandSolder, F.Cu at (124.7, 59.6)
- added C6: 4u7, Capacitor_SMD:C_0201_0603Metric_Pad0.64x0.40mm_HandSolder, F.Cu at (127.1, 48.9)
- added D3: LED, LED_SMD:LED_0201_0603Metric, F.Cu at (123.0, 59.6)
- added IC1: MCP73831T-2ACI_OT, Custom:SOT95P270X145-5N, F.Cu at (121.7, 57.3)
- added J5: Conn_01x02_Pin, Connector_Molex:Molex_CLIK-Mate_502443-0270_1x02-1MP_P2.00mm_Vertical, F.Cu at (124.2, 45.5)
- added PMV33UPE215: ~, Package_TO_SOT_SMD:TSOT-23, F.Cu at (126.4, 57.5)
- added R10: 470, Resistor_SMD:R_0201_0603Metric_Pad0.64x0.40mm_HandSolder, F.Cu at (120.8, 59.6)
- added R9: 2k, Resistor_SMD:R_0201_0603Metric_Pad0.64x0.40mm_HandSolder, F.Cu at (121.7, 54.8)
- D1: value LED -> PMEG2010ER; footprint LED_SMD:LED_0201_0603Metric -> Diode_SMD:Nexperia_CFP3_SOD-123W
- R2: value 1k -> 100k
- moved D1 13.8 mm to (119.7, 50.9), turned to 90 degrees
- moved J3 9.60 mm to (121.5, 61.8)
- moved R1 9.56 mm to (122.2, 53.2), turned to -90 degrees
- moved C2 7.85 mm to (123.7, 50.9)
- moved PS1 7.66 mm to (124.5, 53.5)
- moved L1 7.60 mm to (125.0, 50.9)
- moved C1 7.58 mm to (125.7, 50.9)
- moved R2 6.97 mm to (127.2, 54.6), turned to 180 degrees
Connections:
- C1 pad 2: VBAT -> VSYS
- D1 pad 1: Net-(D1-K) -> VSYS
- PS1 pad 1: VBAT -> VSYS
- PS1 pad 10: VBAT -> VSYS
- PS1 pad 11: VBAT -> VSYS
- PS1 pad 12: VBAT -> VSYS
- PS1 pad 8: VBAT -> VSYS
- PS1 pad 9: VBAT -> VSYS
- R2 pad 1: Net-(U1-~{STDBY}) -> GND
- R2 pad 2: Net-(D2-K) -> VVCC
Routing:
- net MAIN_PWR: track 28.2 -> 2.71 mm, vias 1 -> 0
- net Net-(D2-K): track 23.7 -> 0.00 mm, vias 4 -> 0
- net VVCC: track 23.1 -> 0.00 mm, vias 1 -> 0
- net Net-(D1-K): track 17.8 -> 0.00 mm, vias 2 -> 0
- net VBAT: track 28.3 -> 11.9 mm, vias 2 -> 0
- net LOAD: track 15.7 -> 0.00 mm, vias 1 -> 0
- net Net-(U1-CE): track 13.0 -> 0.00 mm, vias 2 -> 0
- net ADC: track 10.3 -> 0.00 mm
- net Net-(U1-~{CHRG}): track 8.65 -> 0.00 mm, vias 2 -> 0
- net CTRL_SENS: track 7.87 -> 0.00 mm, vias 1 -> 0
- net Net-(U1-~{STDBY}): track 6.76 -> 0.00 mm, vias 2 -> 0
- net Net-(U1-TEMP): track 4.00 -> 0.00 mm
- net Net-(U1-PROG): track 1.83 -> 0.00 mm
- net Net-(PS1-PG): track 1.46 -> 0.00 mm
- net GND: track 1.15 -> 0.00 mm, vias 13 -> 0
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